File: HW/Amp/overture_amp.sch (KiCad schematic (older format))
At the start: 19 parts, among them J1 PWR+, J2 PWR-, J3 IN_L, J4 IN_R, J5 OUT_L, J6 OUT_R, J7 MUTE, U1 LM4766

Commit message: Add V3 (Actually built)
Parts:
- C4: symbol CP -> Device:CP
- J3, J5, J6, J7: symbol CONN_2 -> conn:Conn_01x02
- R1, R3, R5, R6, R7: symbol R -> Device:R
- U1: symbol LM4766 -> suf_poweramp:LM4766
Connections:
- wire segments 53 -> 63
