File: HW/PSU/overture_psu.sch (KiCad schematic (older format))
At the start: 12 parts, among them J1 OUT, J2 IN, J3 LED

Commit message: Add V3 (Actually built)
Parts:
- added C5, C6: 10000uF/50V, Capacitors_ThroughHole:CP_Radial_D35.0mm_P10.00mm_SnapIn, symbol Device:CP
- added C7, C8: 1uF/250V, Capacitors_ThroughHole:C_Rect_L26.5mm_W11.5mm_P22.50mm_MKS4, symbol Device:C
- added J4: OUT2, suf_connector_ncw:CONN_NCW396-03S, symbol conn:Conn_01x03
- added J5: Protect, Connectors_JST:JST_EH_B03B-EH-A_03x2.50mm_Straight, symbol Connector_Generic:Conn_01x03
- C1: footprint C4P_D14 -> Capacitors_ThroughHole:CP_Radial_D35.0mm_P10.00mm_SnapIn; symbol CP -> Device:CP
- C2: renamed from C4; footprint C4P_D14 -> Capacitors_ThroughHole:CP_Radial_D35.0mm_P10.00mm_SnapIn; symbol CP -> Device:CP
- C3: renamed from C2; value 100nF/50V -> 1uF/250V; footprint c_2220 -> Capacitors_ThroughHole:C_Rect_L26.5mm_W11.5mm_P22.50mm_MKS4; symbol C -> Device:C
- C4: renamed from C3; value 100nF/50V -> 1uF/250V; footprint c_2220 -> Capacitors_ThroughHole:C_Rect_L26.5mm_W11.5mm_P22.50mm_MKS4; symbol C -> Device:C
- D1, D2, D3, D4: footprint TO220-2 -> TO_SOT_Packages_THT:TO-220-2_Vertical; symbol DIODE-HEXFRED -> Device:D
- J1: value OUT -> OUT1; footprint CONN_NCW396-02R -> suf_connector_ncw:CONN_NCW396-03S; symbol CONN_2 -> conn:Conn_01x03
- J2: footprint CONN_NCW396-02R -> Terminal_Blocks:TerminalBlock_bornier-4_P5.08mm; symbol CONN_2 -> conn:Conn_01x04
- J3: footprint HDR-2 -> suf_connector_ncw:CONN_NCW254-02S; symbol CONN_2 -> conn:Conn_01x02
- R1: footprint R4 -> Resistors_ThroughHole:R_Axial_DIN0207_L6.3mm_D2.5mm_P10.16mm_Horizontal; symbol R -> Device:R
Connections:
- net labels added: GND
- wire segments 26 -> 62
